File: tuss4470_eval_v1.kicad_sch (KiCad schematic)
At the start: 15 parts, among them IC1 TUSS4470TRTJR, J1 Screw_Terminal_01x02, J2 Conn_01x10_Pin, Q1 2N7002K, T1 42IF102-RC, U1 US_TRANSDUCER

Commit message: v1_complete
Parts:
- added C10: C, symbol Device:C
- added C11: 330p/50V, symbol Device:C
- added C6: 2.2u/160V, Capacitor_SMD:CP_Elec_4x5.3, symbol Device:C_Polarized
- added C7, C8: 2.2n, symbol Device:C
- added C9: 22n, Capacitor_SMD:C_0805_2012Metric, symbol Device:C
- added JP3, JP4: Jumper_2_Small_Bridged, TestPoint:TestPoint_2Pads_Pitch2.54mm_Drill0.8mm, symbol Jumper:Jumper_2_Small_Bridged
- added R2: 200R, Resistor_SMD:R_0805_2012Metric, symbol Device:R
Connections:
- net GNDD is gone; now on net GND: IC1.2 (DGND)
- net GND: now also C10.2, C6.2, C7.2, C8.2, C9.2
- net at T1.3 (PRI_3), U1.1: now also R2.2
- net at IC1.11 (INN): now also JP3.2 (B), JP4.2 (B)
- net at IC1.12 (INP): now also C11.1
- net at IC1.17 (VDRV): now also C6.1
- net at IC1.18 (FLT): now also C7.1, C8.1
- new net: C9.1, JP3.1 (A)
- new net: C11.2, R2.1
- new net: C10.1, JP4.1 (A)
- no-connect marks 2 -> 1
Other:
- moved on the sheet: C1, C2, C3, C4, C5, D1, IC1, J1, J2, JP1, JP2, Q1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
